File: 555_Timer_Clock.kicad_pcb (KiCad board)
At the start: 2 copper layers, 39 x 25 mm, 13 parts, among them J2 CLK_Out, U1 ICM7555xB

Commit message: edit pcb design
Parts:
- added ?: LOGO, CUSTOM FOOTPRINTS:pepe_logo_s, F.Cu at (105.0, 82.2)
- added J1: +5V, my_footprints:Terminal_Block_5mm, F.Cu at (101.5, 72.5)
- added SW1: Trigger, my_footprints:slide_switch_2.54mm, F.Cu at (123.0, 82.0)
- added SW2: RST, my_footprints:tact_switch_5mm, F.Cu at (112.5, 81.5)
Routing:
- net GND: track 0.00 -> 76.6 mm, vias 0 -> 2
- net /Trigger: track 0.00 -> 37.8 mm
- net /+5V: track 0.00 -> 36.8 mm
- net /CLK_Out: track 0.00 -> 25.6 mm, vias 0 -> 1
- net /RST: track 0.00 -> 18.3 mm
- net Net-(U1-DISCH): track 0.00 -> 12.9 mm
- net Net-(D1-K): track 0.00 -> 8.44 mm
- net Net-(U1-CONT): track 0.00 -> 7.46 mm
Other:
- board text added: "DOLOSO GEDALANGA"
